File: pcb/motordriver.kicad_sch (KiCad schematic)
At the start: 52 parts, among them U201 DRV8251/A, U202 INA181A1IDBVR, U203 LM324PWR

Commit message: readme and schematic
Other:
- note added: "DC biasing also active band pass filter fc1, fc2 = 6.39hz, 1591hz gain = 40.16"
- note added: "R205 and R606 should be 10 ohms or less"
- note added: "low pass filter cutoff = 50.36hz"
- note removed: "DC biasing also active band pass filter fc1, fc2 = 63.9hz, 1591hz gain = 40.16"
- note removed: "low pass filter cutoff = 50hz"
- moved on the sheet: R215
