File: pcb/ripplecounter.kicad_pcb (KiCad board)
At the start: 2 copper layers, 82 x 56 mm, 126 parts, among them SW101 PTS636 SM25 SMTR LFS, U101 RPi Pico, U201 DRV8251/A, U202 INA181A1IDBVR, U203 LM324PWR, U301 DRV8251/A, U302 INA181A1IDBVR, U303 LM324PWR

Commit message: readme and schematic
Changed lines of the file:
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@@
     (attr smd)
     (net_tie_pad_groups "1, 2")
-    (fp_text reference "JP102" (at 0 -1.43 90) (layer "F.SilkS")
-        (effects (font (size 1 1) (thickness 0.15)))
+    (fp_text reference "JP102" (at 0 -1.4 90) (layer "F.SilkS")
+        (effects (font (size 0.9 0.7) (thickness 0.12)))
     )
     (fp_text value "~" (at 0 1.43 90) (layer "F.Fab") hide
@@
     (attr smd)
     (net_tie_pad_groups "1, 2")
-    (fp_text reference "JP301" (at 0 -1.43 -90) (layer "F.SilkS")
-        (effects (font (size 1 1) (thickness 0.15)))
+    (fp_text reference "JP301" (at 2.925 0 -90) (layer "F.SilkS")
+        (effects (font (size 0.9 0.7) (thickness 0.12)))
     )
     (fp_text value "~" (at 0 1.43 -90) (layer "F.Fab") hide
@@
     (attr smd)
     (net_tie_pad_groups "1, 2")
-    (fp_text reference "JP105" (at 0 -1.43 -90) (layer "F.SilkS")
-        (effects (font (size 1 1) (thickness 0.15)))
+    (fp_text reference "JP105" (at 0 1.4 -90) (layer "F.SilkS")
+        (effects (font (size 0.9 0.7) (thickness 0.12)))
     )
     (fp_text value "0603_Closed" (at 0 1.43 -90) (layer "F.Fab") hide
@@
     (attr smd)
     (net_tie_pad_groups "1, 2")
-    (fp_text reference "JP108" (at 0 -1.43 90) (layer "F.SilkS")
-        (effects (font (size 1 1) (thickness 0.15)))
+    (fp_text reference "JP108" (at 0 -1.4 90) (layer "F.SilkS")
+        (effects (font (size 0.9 0.7) (thickness 0.12)))
     )
     (fp_text value "~" (at 0 1.43 90) (layer "F.Fab") hide
@@
     (net_tie_pad_groups "1, 2")
     (fp_text reference "JP109" (at 0 -1.43 90) (layer "F.SilkS")
-        (effects (font (size 1 1) (thickness 0.15)))
+        (effects (font (size 0.9 0.7) (thickness 0.12)))
     )
     (fp_text value "~" (at 0 1.43 90) (layer "F.Fab") hide
@@
     (attr smd)
     (net_tie_pad_groups "1, 2")
-    (fp_text reference "JP106" (at 0 -1.43 90) (layer "F.SilkS")
-        (effects (font (size 1 1) (thickness 0.15)))
+    (fp_text reference "JP106" (at 0 -1.4 90) (layer "F.SilkS")
+        (effects (font (size 0.9 0.7) (thickness 0.12)))
     )
     (fp_text value "~" (at 0 1.43 90) (layer "F.Fab") hide
@@
     (attr smd)
     (net_tie_pad_groups "1, 2")
-    (fp_text reference "JP107" (at 0 -1.43 -90) (layer "F.SilkS")
-        (effects (font (size 1 1) (thickness 0.15)))
+    (fp_text reference "JP107" (at 0 1.4 -90) (layer "F.SilkS")
+        (effects (font (size 0.9 0.7) (thickness 0.12)))
     )
     (fp_text value "~" (at 0 1.43 -90) (layer "F.Fab") hide
@@
     (property "ki_keywords" "mounting hole")
     (attr exclude_from_pos_files)
-    (fp_text reference "H101" (at 0 -2.9) (layer "F.SilkS")
-        (effects (font (size 1 1) (thickness 0.15)))
+    (fp_text reference "H101" (at 0 -2.9) (layer "F.SilkS") hide
+        (effects (font (size 0.9 0.7) (thickness 0.12)))
     )
     (fp_text value "~" (at 0 2.9) (layer "F.Fab")
@@
     (attr smd)
     (net_tie_pad_groups "1, 2")
-    (fp_text reference "JP104" (at 0 -1.43 -90) (layer "F.SilkS")
-        (effects (font (size 1 1) (thickness 0.15)))
+    (fp_text reference "JP104" (at 0.0275 1.4 -90) (layer "F.SilkS")
+        (effects (font (size 0.9 0.7) (thickness 0.12)))
     )
     (fp_text value "0603_Closed" (at 0 1.43 -90) (layer "F.Fab") hide
@@
     (attr smd)
     (net_tie_pad_groups "1, 2")
-    (fp_text reference "JP201" (at 0 -1.43 -90) (layer "F.SilkS")
-        (effects (font (size 1 1) (thickness 0.15)))
+    (fp_text reference "JP201" (at 2.875 0 -90) (layer "F.SilkS")
+        (effects (font (size 0.9 0.7) (thickness 0.12)))
     )
     (fp_text value "~" (at 0 1.43 -90) (layer "F.Fab") hide
@@
     (property "ki_keywords" "Solder Jumper SPDT")
     (attr exclude_from_pos_files)
-    (fp_text reference "JP202" (at 0.05 -1.95) (layer "F.SilkS")
-        (effects (font (size 1 1) (thickness 0.15)))
+    (fp_text reference "JP202" (at 3.42375 0.01) (layer "F.SilkS")
+        (effects (font (size 0.9 0.7) (thickness 0.12)))
     )
     (fp_text value "~" (at 0 1.9) (layer "F.Fab")
@@
     (property "ki_keywords" "solder jumper SPST")
     (attr smd)
-    (fp_text reference "JP101" (at 0 -1.43 180) (layer "F.SilkS")
-        (effects (font (size 1 1) (thickness 0.15)))
+    (fp_text reference "JP101" (at 0 1.25 180) (layer "F.SilkS")
+        (effects (font (size 0.9 0.7) (thickness 0.12)))
     )
     (fp_text value "~" (at 0 1.43 180) (layer "F.Fab") hide
@@
     (property "ki_keywords" "Solder Jumper SPDT")
     (attr exclude_from_pos_files)
-    (fp_text reference "JP302" (at 0.05 -1.95) (layer "F.SilkS")
-        (effects (font (size 1 1) (thickness 0.15)))
+    (fp_text reference "JP302" (at 3.39875 0.01) (layer "F.SilkS")
+        (effects (font (size 0.9 0.7) (thickness 0.12)))
     )
     (fp_text value "~" (at 0 1.9) (layer "F.Fab")
@@
     (attr smd)
     (net_tie_pad_groups "1, 2")
-    (fp_text reference "JP103" (at 0 -1.43 90) (layer "F.SilkS")
-        (effects (font (size 1 1) (thickness 0.15)))
+    (fp_text reference "JP103" (at 0 -1.4 90) (layer "F.SilkS")
+        (effects (font (size 0.9 0.7) (thickness 0.12)))
     )
     (fp_text value "~" (at 0 1.43 90) (layer "F.Fab") hide
@@
     (effects (font (size 1 1) (thickness 0.15)) (justify right mirror))
   )
-  (gr_text "JLCJLCJLCJLC" (at 115.25 70.5 90) (layer "F.SilkS")
-    (effects (font (size 1 1) (thickness 0.15)))
-  )
   (gr_text "reset" (at 130.4 88.45 90) (layer "F.SilkS")
     (effects (font (size 1 1) (thickness 0.15)))
@@
     (effects (font (size 1 1) (thickness 0.15)) (justify left))
   )
+  (gr_text "JLCJLCJLCJLC" (at 115.25 70.5 90) (layer "Dwgs.User")
+    (effects (font (size 1 1) (thickness 0.15)))
+  )
   (gr_text "Manufacturing specifications:\n- 2 copper layers\n- size: 82 x 56 mm\n- thickness: 1.6 mm\n- material: FR-4 TG-140+\n- min track width/spacing: 0.2 mm\n- min hole size: 0.3 mm\n- min annular ring size: 0.15mm\n- soldermask: blue\n- silkscreen: white\n- finish: HASL\n- copper: 1 oz\n\nAll mounting holes sized for M2 SHCS/BHCS\n\nDesign by jackw01\nOpen source hardware\nReleased under the CERN-OHL-W V2 license" (at 143.35 93.35) (layer "Cmts.User")
